Commit message: Change package name and add collision visual in urdf file

File: end_effector_control/config/panda_arm_hand.urdf (robot description, URDF)
Before this commit: robot panda, 12 links, 11 joints
Links:
- link panda_link0: geometry collision box size=2.0 2.0 0.05; collision cylinder length=0.03 radius=0.09
