Commit message: Adding environment testing code

File: config/bmi_panda.urdf (robot description, URDF)
Before this commit: robot panda, 12 links, 11 joints
Links:
- link panda_hand: geometry collision mesh filename=package://moveit_resources_panda_description/meshes/collisi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; visual mesh filename=package://moveit_resources_panda_description/meshes/visual/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

File: config/grasp_panda.urdf (robot description, URDF)
Before this commit: robot panda, 12 links, 11 joints
Links:
- link panda_hand: geometry collision mesh filename=package://moveit_resources_panda_description/meshes/collisi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; visual mesh filename=package://moveit_resources_panda_description/meshes/visual/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

File: config/staged_panda.urdf (robot description, URDF)
Before this commit: robot panda, 12 links, 11 joints
Links:
- link panda_hand: geometry collision mesh filename=package://moveit_resources_panda_description/meshes/collisi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; visual mesh filename=package://moveit_resources_panda_description/meshes/visual/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

Commit message: Adding updated environment testing files

File: config/bmi_panda.urdf (robot description, URDF)
Before this commit: robot panda, 12 links, 11 joints
Links:
- link panda_link0: geometry collision box size=2.0 2.0 0.05; collision mesh filename=package://end_effector_control/config/bmi_setup.stl scale=0.001 0.001 0.001
