Commit message: Adding grasping functionality

File: config/staged_panda.urdf (robot description, URDF)
Before this commit: robot panda, 12 links, 11 joints
Joints:
- joint panda_hand_joint: origin xyz=0 0 0.1 rpy=0 0 -0.785398163397 -> xyz=0 0 0.15 rpy=0 0 -0.785398163397

Commit message: Adds various demo and calibration changes
Change Panda joint limits in staged_panda.urdf to the joint limits
specified by the manufacturers
(https://frankaemika.github.io/docs/control_parameters.html). Ideally,
this should lead to the demo not running into joint limits so frequently
anymore.

Shorten planning time from 5 seconds to 2 seconds.

Publish box object of realistic size and offset the location in the
planning scene to account for the fact that the April Tag detection
returns a point on the surface of the box, not in the middle of the box.

Change orientation angle to 0 degrees so panda end effector is verticle
as it tracks the object through the workspace. This allows for easier
joint configurations during object tracking.

Comment out roslib.load_manifest in display_marker_publisher.py. This
line was causing errors when attempting to run the demo and appears
unnecessary.

Edit grasp_test_stationary.py to grip the box used in the demo.

Alter the sample_pose.py script for collecting calibration data. Once
run, it queries the depth camera for the target april tag location -
which should be on the box between the pandas grippers - and stores that
with the location of "panda_link_9" which should be at the desired
location of the target april tag in the URDF. This gives us sim vs real
data that can help us calibrate, the "panda_link_9" location being the
ground truth location of the box in the world frame, and the depth
camera output being the detected location that needs to be calibrated.

Add panda_link_9 in the staged_panda.urdf.

File: config/staged_panda.urdf (robot description, URDF)
Before this commit: robot panda, 12 links, 11 joints
Links:
- added link panda_link9
Joints:
- added joint panda_hand_joint2: type fixed, parent panda_link8, child panda_link9, origin xyz=0 0 0.12 rpy=0 0 -0.785398163397
- joint panda_joint1: limit lower=-2.9671 upper=2.9671 effort=87 velocity=2.3925 -> lower=-2.8973 upper=2.8973 effort=87 velocity=2.3925
- joint panda_joint2: limit lower=-1.8326 upper=1.8326 effort=87 velocity=2.3925 -> lower=-1.7628 upper=1.7628 effort=87 velocity=2.3925
- joint panda_joint3: limit lower=-2.9671 upper=2.9671 effort=87 velocity=2.3925 -> lower=-2.8973 upper=2.8973 effort=87 velocity=2.3925
- joint panda_joint4: limit lower=-3.1416 upper=0.0873 effort=87 velocity=2.3925 -> lower=-3.0718 upper=-0.0698 effort=87 velocity=2.3925
- joint panda_joint5: limit lower=-2.9671 upper=2.9671 effort=12 velocity=2.8710 -> lower=-2.8973 upper=2.8973 effort=12 velocity=2.8710
- joint panda_joint6: limit lower=-0.0873 upper=3.8223 effort=12 velocity=2.8710 -> lower=-0.0175 upper=3.7525 effort=12 velocity=2.8710
- joint panda_joint7: limit lower=-2.9671 upper=2.9671 effort=12 velocity=2.8710 -> lower=-2.8973 upper=2.8973 effort=12 velocity=2.8710

Commit message: Add changes/code for calibration script
Add changes in staged_panda.urdf to specify ground truth calibration
point on the surface of the end-effector where the April tag will be
placed.

Add calibration joint position samples for the calibration script to run
through to gather ground truth vs observed data to build a model with.

Add plan_to_point script to make collection of the joint position
samples easier. The script automates saving a joint position state to a
yaml file.

File: config/staged_panda.urdf (robot description, URDF)
Before this commit: robot panda, 13 links, 12 joints
Links:
- link panda_link9: geometry visual mesh filename=package://moveit_resources_panda_description/meshes/visual/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; visual sphere radius=0.01
Joints:
- joint panda_hand_joint2: origin xyz=0 0 0.12 rpy=0 0 -0.785398163397 -> xyz=0.015 -0.015 0.04 rpy=0 1.5707963267948966 -0.785398163397

Commit message: Debug/implement calibration code
To calibrate:
  `roslaunch panda_moveit_config demo.launch setup:=staged`
  `rosrun camera calibration_test`
  `rosrun end_effector_control calibrate`
Still need to implement target tracking. Currently the target point
being published to point_command by the camera calibration_test node is
the ee april tag position, not the target position.

File: config/staged_panda.urdf (robot description, URDF)
Before this commit: robot panda, 13 links, 12 joints
Links:
- removed link panda_link9
- added link base_april_tag; visual mesh filename=package://moveit_resources_panda_description/meshes/visual/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 scale=1.0 1.0 1.0; visual sphere radius=0.005
- added link ee_april_tag; visual mesh filename=package://moveit_resources_panda_description/meshes/visual/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 scale=0.6 0.6 0.6; visual sphere radius=0.005
Joints:
- removed joint panda_hand_joint2
- added joint april_tag_base_joint: type fixed, parent panda_link0, child base_april_tag, origin xyz=0.06 0.0 0.09 rpy=-1.5707963267948966 0 1.5707963267948966
- added joint ee_april_tag_joint: type fixed, parent panda_link8, child ee_april_tag, origin xyz=0.015 -0.015 0.035 rpy=1.5707963267948966 0 -2.356194490192345

Commit message: Cleanup/update calibration code
Added calibrate_demo.launch file to easily run the automated calibration.
Changed robo_demo.launch to run the new camera package target_publisher
that uses the automated calibration model.
Added go_to_joint_goal node to test planning & execution of joint goals
quickly.
Rename robo_demo.launch to run_demo.launch
Changed show_at_point to show_point node which now takes in a topic
argument when run so it can publish a visualization of a point from any
topic.

File: config/staged_panda.urdf (robot description, URDF)
Before this commit: robot panda, 14 links, 13 joints
Links:
- link ee_april_tag: geometry visual mesh filename=package://moveit_resources_panda_description/meshes/visual/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 scale=0.6 0.6 0.6; visual sphere radius=0.0175
Joints:
- joint ee_april_tag_joint: origin xyz=0.015 -0.015 0.035 rpy=1.5707963267948966 0 -2.356194490192345 -> xyz=0.005 -0.005 0.035 rpy=1.5707963267948966 0 -2.356194490192345

Commit message: Changes for gathering PRT-RRT* results
Change cost norm comparisons (to evaluate path improvements) to 1-norm
in continuous_collision_checker and RRT_star_monitor instead of 2-norm
to align cost calculations to those done in the planner.

Add PRTRRT_star_planner_parent_process node to manage starting the
planner process when an initial goal comes in. (Like what the
RRT_star_monitor node does)

Add utils.py for common functions across nodes (computing costs and near
equality of joint configurations)

Add path_cost_logger and path_recorder for results evaluation &
collection

Add several test interface iterations, v3 is the final test interface
used in the collection of thesis results.

Add rewiring_time_data_collector to collect amount of time it takes on
average to rewire around a node in the root rewiring process. (Just
subscribes to a topic that publishes this information from the PRT-RRT*
planner.

Add files for "change goal test" which sent the panda to an initial
goal, then gave it another goal before the panda had finished executing
the initial goal. These test results are included in the thesis.

Remove visual target ball at extended panda hand joint from
stadged_panda.urdf so thesis document and presentation screenshots
aren't confusing. (random floating red ball doesn't make sense out of
context)

Add automation scripts to automate calling the testing services for
results collection (`automate_testing(_v2).py`).

Add a few tool scripts like `collect_plans` and `path_recorder` to aid
in the development of the data collection scripts.

File: config/staged_panda.urdf (robot description, URDF)
Before this commit: robot panda, 14 links, 13 joints
Links:
- removed link base_april_tag
- removed link ee_april_tag
- link panda_hand: geometry collision mesh filename=package://moveit_resources_panda_description/meshes/collisi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; visual mesh filename=package://moveit_resources_panda_description/meshes/visual/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
Joints:
- removed joint april_tag_base_joint
- removed joint ee_april_tag_joint

Commit message: changes for final results

File: config/staged_panda.urdf (robot description, URDF)
Before this commit: robot panda, 14 links, 13 joints
Links:
- removed link base_april_tag
- removed link ee_april_tag
Joints:
- removed joint april_tag_base_joint
- removed joint ee_april_tag_joint

Commit message: Changes for HW following demo
Uncomment end effector April tag in URDF since it's used in the demo.
Leave the base April Tag commented since it's unused in demo (only
look at the end effector april tag and the target box April Tag).

Add logging output to the screen for the `calibrate` and
`camera_publisher` nodes in the calibrate_demo.launch file.

Increase default control duration to 3 seconds in the
PRTRRT_star_controller.py script for safety. (If the control duration is
lower then the control will have less time to acheive target trajectory
points and as a result the robot will move much faster and more
aggressively).

Add list of zeros to the trajectory point velocity field in the goal
trajectory messages sent to the controller in PRTRRT_star_controller.py.
Without adding these zeros, the Panda shudders during control.

Add some TODO notes in the demo_interface.py file for further demo
improvements.

File: config/staged_panda.urdf (robot description, URDF)
Before this commit: robot panda, 12 links, 11 joints
Links:
- added link ee_april_tag; visual mesh filename=package://moveit_resources_panda_description/meshes/visual/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 scale=0.6 0.6 0.6; visual sphere radius=0.0175
Joints:
- added joint ee_april_tag_joint: type fixed, parent panda_link8, child ee_april_tag, origin xyz=0.005 -0.005 0.035 rpy=1.5707963267948966 0 -2.356194490192345
